Commit message: correct frames and meshes and collisions

File: description/urdf/pupper_v3 world aligned frames.urdf (robot description, URDF)
Before this commit: robot pupper_v3, 13 links, 12 joints
Links:
- link leg_back_l_1: geometry visual mesh filename=../meshes/dae/Leg Assembly For Flanged v26.013.dae scale=1.00000 1.00000 -1.00000
- link leg_front_l_1: geometry visual mesh filename=../meshes/dae/Leg Assembly For Flanged v26.010.dae scale=1.00000 1.00000 -1.00000
Joints:
- joint leg_back_l_1: origin xyz=-0.07500 0.07250 0.00000 rpy=-1.57080 0.00000 0.00000 -> xyz=-0.07500 0.07250 0.00000 rpy=1.57080 0.00000 0.00000
- joint leg_back_l_2: origin xyz=0.00000 0.00000 0.00000 rpy=1.57080 1.57080 -1.57080 -> xyz=0.00000 0.00000 0.00000 rpy=1.49199 -1.57080 -1.49198
- joint leg_back_l_3: origin xyz=0.00000 -0.04940 0.06850 rpy=-0.00000 1.57080 3.14159 -> xyz=0.00000 -0.04940 0.06850 rpy=-0.00000 1.57080 0.00000
- joint leg_front_l_1: origin xyz=0.07500 0.08350 0.00000 rpy=-1.57080 0.00000 0.00000 -> xyz=0.07500 0.08350 0.00000 rpy=1.57080 0.00000 0.00000
- joint leg_front_l_2: origin xyz=0.00000 0.00000 0.00000 rpy=1.57080 1.57080 -1.57080 -> xyz=0.00000 0.00000 0.00000 rpy=1.49199 -1.57080 -1.49198
- joint leg_front_l_3: origin xyz=0.00000 -0.04940 0.06850 rpy=-0.00000 1.57080 3.14159 -> xyz=0.00000 -0.04940 0.06850 rpy=-0.00000 1.57080 0.00000

File: description/urdf/pupper_v3.fixed.urdf (robot description, URDF)
Before this commit: robot pupper_v3, 13 links, 12 joints
Links:
- link base_link: geometry collision box size=0.09014 0.12758 0.25943; visual mesh filename=package://pupper_v3_description/description/meshes/dae/Body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 scale=1.00000 1.00000 1.00000
- link leg_back_l_1: geometry visual mesh filename=package://pupper_v3_description/description/meshes/dae/LegA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 scale=1.00000 1.00000 1.00000
- link leg_back_l_2: geometry collision cylinder length=0.03000 radius=0.02500; visual mesh filename=package://pupper_v3_description/description/meshes/dae/LegA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 scale=1.00000 1.00000 -1.00000
- link leg_back_l_3: geometry collision sphere radius=0.01995; visual mesh filename=package://pupper_v3_description/description/meshes/dae/LegA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 scale=1.00000 1.00000 -1.00000
- link leg_back_r_1: geometry visual mesh filename=package://pupper_v3_description/description/meshes/dae/LegA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 scale=1.00000 1.00000 1.00000
- link leg_back_r_2: geometry collision cylinder length=0.03000 radius=0.02500; visual mesh filename=package://pupper_v3_description/description/meshes/dae/LegA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 scale=1.00000 1.00000 1.00000
- link leg_back_r_3: geometry collision sphere radius=0.01995; visual mesh filename=package://pupper_v3_description/description/meshes/dae/LegA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 scale=1.00000 1.00000 1.00000
- link leg_front_l_1: geometry visual mesh filename=package://pupper_v3_description/description/meshes/dae/LegA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 scale=1.00000 -1.00000 1.00000
- link leg_front_l_2: geometry collision cylinder length=0.03000 radius=0.02500; visual mesh filename=package://pupper_v3_description/description/meshes/dae/LegA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 scale=1.00000 1.00000 -1.00000
- link leg_front_l_3: geometry collision sphere radius=0.01995; visual mesh filename=package://pupper_v3_description/description/meshes/dae/LegA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 scale=1.00000 1.00000 -1.00000
- link leg_front_r_1: geometry visual mesh filename=package://pupper_v3_description/description/meshes/dae/LegA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 scale=1.00000 1.00000 1.00000
- link leg_front_r_2: geometry collision cylinder length=0.03000 radius=0.02500; visual mesh filename=package://pupper_v3_description/description/meshes/dae/LegA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 scale=1.00000 1.00000 1.00000
- link leg_front_r_3: geometry collision sphere radius=0.01995; visual mesh filename=package://pupper_v3_description/description/meshes/dae/LegA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 scale=1.00000 1.00000 1.00000
