Commit message: update masses

File: description/urdf/pupper_v3.fixed.urdf (robot description, URDF)
Before this commit: robot pupper_v3, 13 links, 12 joints
Links:
- link base_link: mass 1.50000 -> 1.506
- link leg_back_l_1: mass 0.15000 -> 0.18000
- link leg_back_l_2: mass 0.15000 -> 0.18600
- link leg_back_r_1: mass 0.15000 -> 0.18000
- link leg_back_r_2: mass 0.15000 -> 0.18600
- link leg_front_l_1: mass 0.15000 -> 0.18000
- link leg_front_l_2: mass 0.15000 -> 0.18600
- link leg_front_r_1: mass 0.15000 -> 0.18000
- link leg_front_r_2: mass 0.15000 -> 0.18600

File: description/urdf/pupper_v3.urdf (robot description, URDF)
Before this commit: robot pupper_v3, 13 links, 12 joints
Links:
- link base_link: mass 1.50000 -> 1.506
- link leg_back_l_1: mass 0.15000 -> 0.18000
- link leg_back_l_2: mass 0.15000 -> 0.18600
- link leg_back_r_1: mass 0.15000 -> 0.18000
- link leg_back_r_2: mass 0.15000 -> 0.18600
- link leg_front_l_1: mass 0.15000 -> 0.18000
- link leg_front_l_2: mass 0.15000 -> 0.18600
- link leg_front_r_1: mass 0.15000 -> 0.18000
- link leg_front_r_2: mass 0.15000 -> 0.18600

Commit message: fix joint limits

File: description/urdf/pupper_v3.fixed.urdf (robot description, URDF)
Before this commit: robot pupper_v3, 13 links, 12 joints
Joints:
- joint leg_back_l_1: limit lower=-1.22000 upper=2.51000 effort=3.00000 velocity=100.00000 -> lower=-2.51000 upper=1.22000 effort=3.00000 velocity=100.00000
- joint leg_back_l_2: limit lower=-0.42000 upper=3.14000 effort=3.00000 velocity=100.00000 -> lower=-3.14000 upper=0.42000 effort=3.00000 velocity=100.00000
- joint leg_back_l_3: limit lower=-2.79000 upper=0.63000 effort=3.00000 velocity=100.00000 -> lower=-0.63000 upper=+2.79000 effort=3.00000 velocity=100.00000
- joint leg_front_l_1: limit lower=-1.22000 upper=2.51000 effort=3.00000 velocity=100.00000 -> lower=-2.51000 upper=1.22000 effort=3.00000 velocity=100.00000
- joint leg_front_l_2: limit lower=-0.42000 upper=3.14000 effort=3.00000 velocity=100.00000 -> lower=-3.14000 upper=0.42000 effort=3.00000 velocity=100.00000
- joint leg_front_l_3: limit lower=-2.79000 upper=0.63000 effort=3.00000 velocity=100.00000 -> lower=-0.63000 upper=+2.79000 effort=3.00000 velocity=100.00000

File: description/urdf/pupper_v3.urdf (robot description, URDF)
Before this commit: robot pupper_v3, 13 links, 12 joints
Joints:
- joint leg_back_l_1: limit lower=-1.22000 upper=2.51000 effort=3.00000 velocity=100.00000 -> lower=-2.51000 upper=1.22000 effort=3.00000 velocity=100.00000
- joint leg_back_l_2: limit lower=-0.42000 upper=3.14000 effort=3.00000 velocity=100.00000 -> lower=-3.14000 upper=0.42000 effort=3.00000 velocity=100.00000
- joint leg_back_l_3: limit lower=-2.79000 upper=0.63000 effort=3.00000 velocity=100.00000 -> lower=-0.63000 upper=+2.79000 effort=3.00000 velocity=100.00000
- joint leg_front_l_1: limit lower=-1.22000 upper=2.51000 effort=3.00000 velocity=100.00000 -> lower=-2.51000 upper=1.22000 effort=3.00000 velocity=100.00000
- joint leg_front_l_2: limit lower=-0.42000 upper=3.14000 effort=3.00000 velocity=100.00000 -> lower=-3.14000 upper=0.42000 effort=3.00000 velocity=100.00000
- joint leg_front_l_3: limit lower=-2.79000 upper=0.63000 effort=3.00000 velocity=100.00000 -> lower=-0.63000 upper=+2.79000 effort=3.00000 velocity=100.00000
