Commit message: Update URDF and add Blender file containing Phobos model

File: description/urdf/pupper_v3.urdf (robot description, URDF)
Before this commit: robot pupper_v3, 13 links, 12 joints
Links:
- link base_link: mass 1.0 -> 1.0000000; geometry collision box size=0.0901404 0.1275797 0.2594327; visual mesh filename=../meshes/dae/Body V4 v70.001.dae scale=1.0000000 1.0000000 1.0000000
- link leg_back_l_1: mass 0.2 -> 0.1500000; geometry visual mesh filename=../meshes/dae/Leg Assembly For Flanged v26.013.dae scale=-1.0000000 -1.0000000 -1.0000000
- link leg_back_l_2: mass 0.2 -> 0.1500000; geometry collision cylinder length=0.0300000 radius=0.0250000; visual mesh filename=../meshes/dae/Leg Assembly For Flanged v26.014.dae scale=-1.0000000 -1.0000000 -1.0000000
- link leg_back_l_3: mass 0.045 -> 0.0500000; geometry collision sphere radius=0.0199511; visual mesh filename=../meshes/dae/Leg Assembly For Flanged v26.015.dae scale=-1.0000000 -1.0000000 -1.0000000
- link leg_back_r_1: mass 0.2 -> 0.1500000; geometry visual mesh filename=../meshes/dae/Leg Assembly For Flanged v26.005.dae scale=1.0000000 1.0000000 1.0000000
- link leg_back_r_2: mass 0.2 -> 0.1500000; geometry collision cylinder length=0.0300000 radius=0.0250000; visual mesh filename=../meshes/dae/Leg Assembly For Flanged v26.006.dae scale=1.0000000 1.0000000 1.0000000
- link leg_back_r_3: mass 0.045 -> 0.0500000; geometry collision sphere radius=0.0199511; visual mesh filename=../meshes/dae/Leg Assembly For Flanged v26.007.dae scale=1.0000000 1.0000000 1.0000000
- link leg_front_l_1: mass 0.2 -> 0.1500000; geometry visual mesh filename=../meshes/dae/Leg Assembly For Flanged v26.010.dae scale=-1.0000000 -1.0000000 -1.0000000
- link leg_front_l_2: mass 0.2 -> 0.1500000; geometry collision cylinder length=0.0300000 radius=0.0250000; visual mesh filename=../meshes/dae/Leg Assembly For Flanged v26.011.dae scale=-1.0000000 -1.0000000 -1.0000000
- link leg_front_l_3: mass 0.045 -> 0.0500000; geometry collision sphere radius=0.0199511; visual mesh filename=../meshes/dae/Leg Assembly For Flanged v26.012.dae scale=-1.0000000 -1.0000000 -1.0000000
- link leg_front_r_1: mass 0.2 -> 0.1500000; geometry visual mesh filename=../meshes/dae/Leg Assembly For Flanged v26.001.dae scale=1.0000000 1.0000000 1.0000000
- link leg_front_r_2: mass 0.2 -> 0.1500000; geometry collision cylinder length=0.0300000 radius=0.0250000; visual mesh filename=../meshes/dae/Leg Assembly For Flanged v26.002.dae scale=1.0000000 1.0000000 1.0000000
- link leg_front_r_3: mass 0.045 -> 0.0500000; geometry collision sphere radius=0.0199511; visual mesh filename=../meshes/dae/Leg Assembly For Flanged v26.003.dae scale=1.0000000 1.0000000 1.0000000
Joints:
- joint leg_back_l_1: axis 0 0 1.0 -> 0.0000000 0.0000000 1.0000000; limit lower=-2.0944 upper=1.22173 effort=3.7 velocity=47.12389 -> lower=-1.2200000 upper=2.5100000 effort=3.0000000 velocity=100.0000000; origin xyz=-0.075 0.05 0 rpy=-1.5708 0 0 -> xyz=-0.0750000 0.0725000 0.0000000 rpy=3.1415927 0.0000000 0.0000000
- joint leg_back_l_2: axis 0 0 -1.0 -> 0.0000000 0.0000000 1.0000000; limit lower=-0.87266 upper=0.5236 effort=3.7 velocity=47.12389 -> lower=-0.4200000 upper=3.1400001 effort=3.0000000 velocity=100.0000000; origin xyz=0 0 0.034 rpy=1.5708 0 1.5708 -> xyz=0.0000000 0.0000000 0.0000000 rpy=1.4919850 -1.5707962 -1.4919850
- joint leg_back_l_3: axis 0 0 -1.0 -> 0.0000000 0.0000000 1.0000000; limit lower=-0.82903 upper=3.05433 effort=3.7 velocity=47.12389 -> lower=-2.7900000 upper=0.6300000 effort=3.0000000 velocity=100.0000000; origin xyz=0.0515 0 -0.07 rpy=1.5708 2.26893 0 -> xyz=0.0000000 -0.0494000 0.0685000 rpy=-0.0000002 1.5707963 0.0000000
- joint leg_back_r_1: axis 0 0 1.0 -> 0.0000000 0.0000000 1.0000000; limit lower=-1.22173 upper=2.0944 effort=3.7 velocity=47.12389 -> lower=-1.2200000 upper=2.5100000 effort=3.0000000 velocity=100.0000000; origin xyz=-0.075 -0.05 0 rpy=1.5708 0 0 -> xyz=-0.0750000 -0.0725000 0.0000000 rpy=1.5707963 0.0000000 0.0000000
- joint leg_back_r_2: axis 0 0 1.0 -> 0.0000000 0.0000000 1.0000000; limit lower=-0.5236 upper=0.87266 effort=3.7 velocity=47.12389 -> lower=-0.4200000 upper=3.1400001 effort=3.0000000 velocity=100.0000000; origin xyz=0 0 0.034 rpy=-1.5708 0 1.5708 -> xyz=0.0000000 0.0000000 0.0000000 rpy=1.4919850 -1.5707962 -1.4919850
- joint leg_back_r_3: axis 0 0 1.0 -> 0.0000000 0.0000000 1.0000000; limit lower=-3.05433 upper=0.82903 effort=3.7 velocity=47.12389 -> lower=-2.7900000 upper=0.6300000 effort=3.0000000 velocity=100.0000000; origin xyz=-0.0515 0 0.07 rpy=1.5708 2.26893 0 -> xyz=0.0000000 -0.0494000 0.0685000 rpy=-0.0000002 1.5707963 0.0000000
- joint leg_front_l_1: axis 0 0 1.0 -> 0.0000000 0.0000000 1.0000000; limit lower=-2.0944 upper=1.22173 effort=3.7 velocity=47.12389 -> lower=-1.2200000 upper=2.5100000 effort=3.0000000 velocity=100.0000000; origin xyz=0.075 0.05 0 rpy=-1.5708 0 0 -> xyz=0.0750000 0.0835000 0.0000000 rpy=3.1415927 0.0000000 0.0000000
- joint leg_front_l_2: axis 0 0 -1.0 -> 0.0000000 0.0000000 1.0000000; limit lower=-0.87266 upper=0.5236 effort=3.7 velocity=47.12389 -> lower=-0.4200000 upper=3.1400001 effort=3.0000000 velocity=100.0000000; origin xyz=0 0 0.034 rpy=1.5708 0 1.5708 -> xyz=0.0000000 0.0000000 0.0000000 rpy=1.4919850 -1.5707962 -1.4919850
- joint leg_front_l_3: axis 0 0 -1.0 -> 0.0000000 0.0000000 1.0000000; limit lower=-0.82903 upper=3.05433 effort=3.7 velocity=47.12389 -> lower=-2.7900000 upper=0.6300000 effort=3.0000000 velocity=100.0000000; origin xyz=0.0515 0 -0.07 rpy=1.5708 2.26893 0 -> xyz=0.0000000 -0.0494000 0.0685000 rpy=-0.0000002 1.5707963 0.0000000
- joint leg_front_r_1: axis 0 0 1.0 -> 0.0000000 0.0000000 1.0000000; limit lower=-1.22173 upper=2.0944 effort=3.7 velocity=47.12389 -> lower=-1.2200000 upper=2.5100000 effort=3.0000000 velocity=100.0000000; origin xyz=0.075 -0.05 0 rpy=1.5708 0 0 -> xyz=0.0750000 -0.0835000 0.0000000 rpy=1.5707963 0.0000000 0.0000000
- joint leg_front_r_2: axis 0 0 1.0 -> 0.0000000 0.0000000 1.0000000; limit lower=-0.5236 upper=0.87266 effort=3.7 velocity=47.12389 -> lower=-0.4200000 upper=3.1400001 effort=3.0000000 velocity=100.0000000; origin xyz=0 0 0.034 rpy=-1.5708 0 1.5708 -> xyz=0.0000000 0.0000000 0.0000000 rpy=1.4919850 -1.5707962 -1.4919850
- joint leg_front_r_3: axis 0 0 1.0 -> 0.0000000 0.0000000 1.0000000; limit lower=-3.05433 upper=0.82903 effort=3.7 velocity=47.12389 -> lower=-2.7900000 upper=0.6300000 effort=3.0000000 velocity=100.0000000; origin xyz=-0.0515 0 0.07 rpy=1.5708 2.26893 0 -> xyz=0.0000000 -0.0494000 0.0685000 rpy=-0.0000002 1.5707963 0.0000000

Commit message: Update body inertias

File: description/urdf/pupper_v3.urdf (robot description, URDF)
Before this commit: robot pupper_v3, 13 links, 12 joints
Links:
- link base_link: mass 1.0000000 -> 1.50000; geometry collision box size=0.09014 0.12758 0.25943; visual mesh filename=../meshes/dae/Body V4 v70.001.dae scale=1.00000 1.00000 1.00000
- link leg_back_l_1: mass 0.1500000 -> 0.15000; geometry visual mesh filename=../meshes/dae/Leg Assembly For Flanged v26.013.dae scale=-1.00000 -1.00000 -1.00000
- link leg_back_l_2: mass 0.1500000 -> 0.15000; geometry collision cylinder length=0.03000 radius=0.02500; visual mesh filename=../meshes/dae/Leg Assembly For Flanged v26.014.dae scale=-1.00000 -1.00000 -1.00000
- link leg_back_l_3: mass 0.0500000 -> 0.05000; geometry collision sphere radius=0.01995; visual mesh filename=../meshes/dae/Leg Assembly For Flanged v26.015.dae scale=-1.00000 -1.00000 -1.00000
- link leg_back_r_1: mass 0.1500000 -> 0.15000; geometry visual mesh filename=../meshes/dae/Leg Assembly For Flanged v26.005.dae scale=1.00000 1.00000 1.00000
- link leg_back_r_2: mass 0.1500000 -> 0.15000; geometry collision cylinder length=0.03000 radius=0.02500; visual mesh filename=../meshes/dae/Leg Assembly For Flanged v26.006.dae scale=1.00000 1.00000 1.00000
- link leg_back_r_3: mass 0.0500000 -> 0.05000; geometry collision sphere radius=0.01995; visual mesh filename=../meshes/dae/Leg Assembly For Flanged v26.007.dae scale=1.00000 1.00000 1.00000
- link leg_front_l_1: mass 0.1500000 -> 0.15000; geometry visual mesh filename=../meshes/dae/Leg Assembly For Flanged v26.010.dae scale=-1.00000 -1.00000 -1.00000
- link leg_front_l_2: mass 0.1500000 -> 0.15000; geometry collision cylinder length=0.03000 radius=0.02500; visual mesh filename=../meshes/dae/Leg Assembly For Flanged v26.011.dae scale=-1.00000 -1.00000 -1.00000
- link leg_front_l_3: mass 0.0500000 -> 0.05000; geometry collision sphere radius=0.01995; visual mesh filename=../meshes/dae/Leg Assembly For Flanged v26.012.dae scale=-1.00000 -1.00000 -1.00000
- link leg_front_r_1: mass 0.1500000 -> 0.15000; geometry visual mesh filename=../meshes/dae/Leg Assembly For Flanged v26.001.dae scale=1.00000 1.00000 1.00000
- link leg_front_r_2: mass 0.1500000 -> 0.15000; geometry collision cylinder length=0.03000 radius=0.02500; visual mesh filename=../meshes/dae/Leg Assembly For Flanged v26.002.dae scale=1.00000 1.00000 1.00000
- link leg_front_r_3: mass 0.0500000 -> 0.05000; geometry collision sphere radius=0.01995; visual mesh filename=../meshes/dae/Leg Assembly For Flanged v26.003.dae scale=1.00000 1.00000 1.00000
Joints:
- joint leg_back_l_1: axis 0.0000000 0.0000000 1.0000000 -> 0.00000 0.00000 1.00000; limit lower=-1.2200000 upper=2.5100000 effort=3.0000000 velocity=100.0000000 -> lower=-1.22000 upper=2.51000 effort=3.00000 velocity=100.00000; origin xyz=-0.0750000 0.0725000 0.0000000 rpy=3.1415927 0.0000000 0.0000000 -> xyz=-0.07500 0.07250 0.00000 rpy=3.14159 0.00000 0.00000
- joint leg_back_l_2: axis 0.0000000 0.0000000 1.0000000 -> 0.00000 0.00000 1.00000; limit lower=-0.4200000 upper=3.1400001 effort=3.0000000 velocity=100.0000000 -> lower=-0.42000 upper=3.14000 effort=3.00000 velocity=100.00000; origin xyz=0.0000000 0.0000000 0.0000000 rpy=1.4919850 -1.5707962 -1.4919850 -> xyz=0.00000 0.00000 0.00000 rpy=1.49199 -1.57080 -1.49198
- joint leg_back_l_3: axis 0.0000000 0.0000000 1.0000000 -> 0.00000 0.00000 1.00000; limit lower=-2.7900000 upper=0.6300000 effort=3.0000000 velocity=100.0000000 -> lower=-2.79000 upper=0.63000 effort=3.00000 velocity=100.00000; origin xyz=0.0000000 -0.0494000 0.0685000 rpy=-0.0000002 1.5707963 0.0000000 -> xyz=0.00000 -0.04940 0.06850 rpy=-0.00000 1.57080 0.00000
- joint leg_back_r_1: axis 0.0000000 0.0000000 1.0000000 -> 0.00000 0.00000 1.00000; limit lower=-1.2200000 upper=2.5100000 effort=3.0000000 velocity=100.0000000 -> lower=-1.22000 upper=2.51000 effort=3.00000 velocity=100.00000; origin xyz=-0.0750000 -0.0725000 0.0000000 rpy=1.5707963 0.0000000 0.0000000 -> xyz=-0.07500 -0.07250 0.00000 rpy=1.57080 0.00000 0.00000
- joint leg_back_r_2: axis 0.0000000 0.0000000 1.0000000 -> 0.00000 0.00000 1.00000; limit lower=-0.4200000 upper=3.1400001 effort=3.0000000 velocity=100.0000000 -> lower=-0.42000 upper=3.14000 effort=3.00000 velocity=100.00000; origin xyz=0.0000000 0.0000000 0.0000000 rpy=1.4919850 -1.5707962 -1.4919850 -> xyz=0.00000 0.00000 0.00000 rpy=1.49199 -1.57080 -1.49198
- joint leg_back_r_3: axis 0.0000000 0.0000000 1.0000000 -> 0.00000 0.00000 1.00000; limit lower=-2.7900000 upper=0.6300000 effort=3.0000000 velocity=100.0000000 -> lower=-2.79000 upper=0.63000 effort=3.00000 velocity=100.00000; origin xyz=0.0000000 -0.0494000 0.0685000 rpy=-0.0000002 1.5707963 0.0000000 -> xyz=0.00000 -0.04940 0.06850 rpy=-0.00000 1.57080 0.00000
- joint leg_front_l_1: axis 0.0000000 0.0000000 1.0000000 -> 0.00000 0.00000 1.00000; limit lower=-1.2200000 upper=2.5100000 effort=3.0000000 velocity=100.0000000 -> lower=-1.22000 upper=2.51000 effort=3.00000 velocity=100.00000; origin xyz=0.0750000 0.0835000 0.0000000 rpy=3.1415927 0.0000000 0.0000000 -> xyz=0.07500 0.08350 0.00000 rpy=3.14159 0.00000 0.00000
- joint leg_front_l_2: axis 0.0000000 0.0000000 1.0000000 -> 0.00000 0.00000 1.00000; limit lower=-0.4200000 upper=3.1400001 effort=3.0000000 velocity=100.0000000 -> lower=-0.42000 upper=3.14000 effort=3.00000 velocity=100.00000; origin xyz=0.0000000 0.0000000 0.0000000 rpy=1.4919850 -1.5707962 -1.4919850 -> xyz=0.00000 0.00000 0.00000 rpy=1.49199 -1.57080 -1.49198
- joint leg_front_l_3: axis 0.0000000 0.0000000 1.0000000 -> 0.00000 0.00000 1.00000; limit lower=-2.7900000 upper=0.6300000 effort=3.0000000 velocity=100.0000000 -> lower=-2.79000 upper=0.63000 effort=3.00000 velocity=100.00000; origin xyz=0.0000000 -0.0494000 0.0685000 rpy=-0.0000002 1.5707963 0.0000000 -> xyz=0.00000 -0.04940 0.06850 rpy=-0.00000 1.57080 0.00000
- joint leg_front_r_1: axis 0.0000000 0.0000000 1.0000000 -> 0.00000 0.00000 1.00000; limit lower=-1.2200000 upper=2.5100000 effort=3.0000000 velocity=100.0000000 -> lower=-1.22000 upper=2.51000 effort=3.00000 velocity=100.00000; origin xyz=0.0750000 -0.0835000 0.0000000 rpy=1.5707963 0.0000000 0.0000000 -> xyz=0.07500 -0.08350 0.00000 rpy=1.57080 0.00000 0.00000
- joint leg_front_r_2: axis 0.0000000 0.0000000 1.0000000 -> 0.00000 0.00000 1.00000; limit lower=-0.4200000 upper=3.1400001 effort=3.0000000 velocity=100.0000000 -> lower=-0.42000 upper=3.14000 effort=3.00000 velocity=100.00000; origin xyz=0.0000000 0.0000000 0.0000000 rpy=1.4919850 -1.5707962 -1.4919850 -> xyz=0.00000 0.00000 0.00000 rpy=1.49199 -1.57080 -1.49198
- joint leg_front_r_3: axis 0.0000000 0.0000000 1.0000000 -> 0.00000 0.00000 1.00000; limit lower=-2.7900000 upper=0.6300000 effort=3.0000000 velocity=100.0000000 -> lower=-2.79000 upper=0.63000 effort=3.00000 velocity=100.00000; origin xyz=0.0000000 -0.0494000 0.0685000 rpy=-0.0000002 1.5707963 0.0000000 -> xyz=0.00000 -0.04940 0.06850 rpy=-0.00000 1.57080 0.00000

Commit message: add stls

File: description/urdf/pupper_v3.urdf (robot description, URDF)
Before this commit: robot pupper_v3, 13 links, 12 joints
Links:
- link base_link: mass 1.506 -> 1.50000; geometry collision box size=0.09014 0.12758 0.25943; visual mesh filename=../meshes/stl/Body V4 v70.001.stl scale=1.00000 1.00000 1.00000
- link leg_back_l_1: mass 0.18000 -> 0.15000; geometry visual mesh filename=../meshes/stl/Leg Assembly For Flanged v26.013.stl scale=-1.00000 -1.00000 -1.00000
- link leg_back_l_2: mass 0.18600 -> 0.15000; geometry collision cylinder length=0.03000 radius=0.02500; visual mesh filename=../meshes/stl/Leg Assembly For Flanged v26.014.stl scale=-1.00000 -1.00000 -1.00000
- link leg_back_l_3: geometry collision sphere radius=0.01995; visual mesh filename=../meshes/stl/Leg Assembly For Flanged v26.015.stl scale=-1.00000 -1.00000 -1.00000
- link leg_back_r_1: mass 0.18000 -> 0.15000; geometry visual mesh filename=../meshes/stl/Leg Assembly For Flanged v26.005.stl scale=1.00000 1.00000 1.00000
- link leg_back_r_2: mass 0.18600 -> 0.15000; geometry collision cylinder length=0.03000 radius=0.02500; visual mesh filename=../meshes/stl/Leg Assembly For Flanged v26.006.stl scale=1.00000 1.00000 1.00000
- link leg_back_r_3: geometry collision sphere radius=0.01995; visual mesh filename=../meshes/stl/Leg Assembly For Flanged v26.007.stl scale=1.00000 1.00000 1.00000
- link leg_front_l_1: mass 0.18000 -> 0.15000; geometry visual mesh filename=../meshes/stl/Leg Assembly For Flanged v26.010.stl scale=-1.00000 -1.00000 -1.00000
- link leg_front_l_2: mass 0.18600 -> 0.15000; geometry collision cylinder length=0.03000 radius=0.02500; visual mesh filename=../meshes/stl/Leg Assembly For Flanged v26.011.stl scale=-1.00000 -1.00000 -1.00000
- link leg_front_l_3: geometry collision sphere radius=0.01995; visual mesh filename=../meshes/stl/Leg Assembly For Flanged v26.012.stl scale=-1.00000 -1.00000 -1.00000
- link leg_front_r_1: mass 0.18000 -> 0.15000; geometry visual mesh filename=../meshes/stl/Leg Assembly For Flanged v26.001.stl scale=1.00000 1.00000 1.00000
- link leg_front_r_2: mass 0.18600 -> 0.15000; geometry collision cylinder length=0.03000 radius=0.02500; visual mesh filename=../meshes/stl/Leg Assembly For Flanged v26.002.stl scale=1.00000 1.00000 1.00000
- link leg_front_r_3: geometry collision sphere radius=0.01995; visual mesh filename=../meshes/stl/Leg Assembly For Flanged v26.003.stl scale=1.00000 1.00000 1.00000
Joints:
- joint leg_back_l_1: limit lower=-2.51000 upper=1.22000 effort=3.00000 velocity=100.00000 -> lower=-1.22000 upper=2.51000 effort=3.00000 velocity=100.00000; origin xyz=-0.07500 0.07250 0.00000 rpy=-1.57080 0.00000 0.00000 -> xyz=-0.07500 0.07250 0.00000 rpy=3.14159 0.00000 0.00000
- joint leg_back_l_2: limit lower=-3.14000 upper=0.42000 effort=3.00000 velocity=100.00000 -> lower=-0.42000 upper=3.14000 effort=3.00000 velocity=100.00000; origin xyz=0.00000 0.00000 0.00000 rpy=1.57080 1.57080 -1.57080 -> xyz=0.00000 0.00000 0.00000 rpy=1.49199 -1.57080 -1.49198
- joint leg_back_l_3: limit lower=-0.63000 upper=+2.79000 effort=3.00000 velocity=100.00000 -> lower=-2.79000 upper=0.63000 effort=3.00000 velocity=100.00000; origin xyz=0.00000 -0.04940 0.06850 rpy=-0.00000 1.57080 3.14159 -> xyz=0.00000 -0.04940 0.06850 rpy=-0.00000 1.57080 0.00000
- joint leg_front_l_1: limit lower=-2.51000 upper=1.22000 effort=3.00000 velocity=100.00000 -> lower=-1.22000 upper=2.51000 effort=3.00000 velocity=100.00000; origin xyz=0.07500 0.08350 0.00000 rpy=-1.57080 0.00000 0.00000 -> xyz=0.07500 0.08350 0.00000 rpy=3.14159 0.00000 0.00000
- joint leg_front_l_2: limit lower=-3.14000 upper=0.42000 effort=3.00000 velocity=100.00000 -> lower=-0.42000 upper=3.14000 effort=3.00000 velocity=100.00000; origin xyz=0.00000 0.00000 0.00000 rpy=1.57080 1.57080 -1.57080 -> xyz=0.00000 0.00000 0.00000 rpy=1.49199 -1.57080 -1.49198
- joint leg_front_l_3: limit lower=-0.63000 upper=+2.79000 effort=3.00000 velocity=100.00000 -> lower=-2.79000 upper=0.63000 effort=3.00000 velocity=100.00000; origin xyz=0.00000 -0.04940 0.06850 rpy=-0.00000 1.57080 3.14159 -> xyz=0.00000 -0.04940 0.06850 rpy=-0.00000 1.57080 0.00000
