Commit message: use stls for compatibility with mujoco

File: description/urdf/pupper_v3.edited.fixed.urdf (robot description, URDF)
Before this commit: robot pupper_v3, 13 links, 12 joints
Links:
- link base_link: geometry collision box size=0.09014 0.12758 0.25943; visual mesh filename=package://pupper_v3_description/description/meshes/stl/Body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 scale=1.00000 1.00000 1.00000
- link leg_back_l_1: geometry visual mesh filename=package://pupper_v3_description/description/meshes/stl/LegA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 scale=1.00000 -1.00000 1.00000
- link leg_back_l_2: geometry collision cylinder length=0.03000 radius=0.02500; visual mesh filename=package://pupper_v3_description/description/meshes/stl/LegA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 scale=1.00000 1.00000 -1.00000
- link leg_back_l_3: geometry collision sphere radius=0.01995; visual mesh filename=package://pupper_v3_description/description/meshes/stl/LegA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 scale=1.00000 1.00000 -1.00000
- link leg_back_r_1: geometry visual mesh filename=package://pupper_v3_description/description/meshes/stl/LegA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 scale=1.00000 1.00000 1.00000
- link leg_back_r_2: geometry collision cylinder length=0.03000 radius=0.02500; visual mesh filename=package://pupper_v3_description/description/meshes/stl/LegA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 scale=1.00000 1.00000 1.00000
- link leg_back_r_3: geometry collision sphere radius=0.01995; visual mesh filename=package://pupper_v3_description/description/meshes/stl/LegA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 scale=1.00000 1.00000 1.00000
- link leg_front_l_1: geometry visual mesh filename=package://pupper_v3_description/description/meshes/stl/LegA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 scale=1.00000 -1.00000 1.00000
- link leg_front_l_2: geometry collision cylinder length=0.03000 radius=0.02500; visual mesh filename=package://pupper_v3_description/description/meshes/stl/LegA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 scale=1.00000 1.00000 -1.00000
- link leg_front_l_3: geometry collision sphere radius=0.01995; visual mesh filename=package://pupper_v3_description/description/meshes/stl/LegA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 scale=1.00000 1.00000 -1.00000
- link leg_front_r_1: geometry visual mesh filename=package://pupper_v3_description/description/meshes/stl/LegA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 scale=1.00000 1.00000 1.00000
- link leg_front_r_2: geometry collision cylinder length=0.03000 radius=0.02500; visual mesh filename=package://pupper_v3_description/description/meshes/stl/LegA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 scale=1.00000 1.00000 1.00000
- link leg_front_r_3: geometry collision sphere radius=0.01995; visual mesh filename=package://pupper_v3_description/description/meshes/stl/LegA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 scale=1.00000 1.00000 1.00000

File: description/urdf/pupper_v3.edited.urdf (robot description, URDF)
Before this commit: robot pupper_v3, 13 links, 12 joints
Links:
- link leg_back_l_1: geometry visual mesh filename=../meshes/dae/Leg Assembly For Flanged v26.013.dae scale=1.00000 -1.00000 1.00000

Commit message: Add conversion scripts. Make fixes. Update README

File: description/urdf/pupper_v3.edited.fixed.urdf (robot description, URDF)
Before this commit: robot pupper_v3, 13 links, 12 joints
Links:
- added link world
Joints:
- added joint world_to_body: type floating, parent world, child base_link
- joint leg_back_l_3: limit lower=-0.63000 upper=+2.79000 effort=3.00000 velocity=100.00000 -> lower=-0.71000 upper=+2.79000 effort=3.00000 velocity=100.00000
- joint leg_back_r_3: limit lower=-2.79000 upper=0.63000 effort=3.00000 velocity=100.00000 -> lower=-2.79000 upper=0.71000 effort=3.00000 velocity=100.00000
- joint leg_front_l_3: limit lower=-0.63000 upper=+2.79000 effort=3.00000 velocity=100.00000 -> lower=-0.71000 upper=+2.79000 effort=3.00000 velocity=100.00000
- joint leg_front_r_3: limit lower=-2.79000 upper=0.63000 effort=3.00000 velocity=100.00000 -> lower=-2.79000 upper=0.71000 effort=3.00000 velocity=100.00000

File: description/urdf/pupper_v3.edited.urdf (robot description, URDF)
Before this commit: robot pupper_v3, 13 links, 12 joints
Joints:
- joint leg_back_l_3: limit lower=-0.63000 upper=+2.79000 effort=3.00000 velocity=100.00000 -> lower=-0.71000 upper=+2.79000 effort=3.00000 velocity=100.00000
- joint leg_back_r_3: limit lower=-2.79000 upper=0.63000 effort=3.00000 velocity=100.00000 -> lower=-2.79000 upper=0.71000 effort=3.00000 velocity=100.00000
- joint leg_front_l_3: limit lower=-0.63000 upper=+2.79000 effort=3.00000 velocity=100.00000 -> lower=-0.71000 upper=+2.79000 effort=3.00000 velocity=100.00000
- joint leg_front_r_3: limit lower=-2.79000 upper=0.63000 effort=3.00000 velocity=100.00000 -> lower=-2.79000 upper=0.71000 effort=3.00000 velocity=100.00000
