Commit message: update components max kp and effort

File: description/components.xacro (robot description, xacro)
@@ -2,4 +2,142 @@
 <robot xmlns:xacro="http://www.ros.org/wiki/xacro">
     <xacro:macro name="define_components">
+        <joint name="leg_front_l_1">
+            <param name="can_channel">1</param>
+            <param name="can_id">1</param>
+            <param name="homing_stage">2</param>
+            <param name="homing_velocity">1.0</param>
+            <param name="homed_position">1.22</param>
+            <param name="homing_kp">5.5</param>
+            <param name="homing_kd">0.2</param>
+            <param name="homing_torque_threshold">2.0</param>
+            <param name="position_min">-1.0</param>
+            <param name="position_max">1.0</param>
+            <param name="velocity_max">1.0</param>
+            <param name="effort_max">3.0</param>
+            <param name="kp_max">10.0</param>
+            <param name="kd_max">1.0</param>
+            <command_interface name="position"/>
+            <command_interface name="velocity"/>
+            <command_interface name="effort"/>
+            <command_interface name="kp"/>
+            <command_interface name="kd"/>
+            <state_interface name="position"/>
+            <state_interface name="velocity"/>
+        </joint>
+        <joint name="leg_front_l_2">
+            <param name="can_channel">1</param>
+            <param name="can_id">2</param>
+            <param name="homing_stage">1</param>
+            <param name="homing_velocity">1.0</param>
+            <param name="homed_position">0.42</param>
+            <param name="homing_kp">5.5</param>
+            <param name="homing_kd">0.2</param>
+            <param name="homing_torque_threshold">2.0</param>
+            <param name="position_min">-1.0</param>
+            <param name="position_max">1.0</param>
+            <param name="velocity_max">1.0</param>
+            <param name="effort_max">3.0</param>
+            <param name="kp_max">10.0</param>
+            <param name="kd_max">1.0</param>
+            <command_interface name="position"/>
+            <command_interface name="velocity"/>
+            <command_interface name="effort"/>
+            <command_interface name="kp"/>
+            <command_interface name="kd"/>
+            <state_interface name="position"/>
+            <state_interface name="velocity"/>
+        </joint>
+        <joint name="leg_front_l_3">
+            <param name="can_channel">1</param>
+            <param name="can_id">3</param>
+            <param name="homing_stage">0</param>
+            <param name="homing_velocity">-1.0</param>
+            <param name="homed_position">-0.62</param>
+            <param name="homing_kp">5.5</param>
+            <param name="homing_kd">0.2</param>
+            <param name="homing_torque_threshold">2.0</param>
+            <param name="position_min">-1.0</param>
+            <param name="position_max">1.0</param>
+            <param name="velocity_max">1.0</param>
+            <param name="effort_max">3.0</param>
+            <param name="kp_max">10.0</param>
+            <param name="kd_max">1.0</param>
+            <command_interface name="position"/>
+            <command_interface name="velocity"/>
+            <command_interface name="effort"/>
+            <command_interface name="kp"/>
+            <command_interface name="kd"/>
+            <state_interface name="position"/>
+            <state_interface name="velocity"/>
+        </joint>
+        <joint name="leg_back_l_1">
+            <param name="can_channel">3</param>
+            <param name="can_id">1</param>
+            <param name="homing_stage">2</param>
+            <param name="homing_velocity">1.0</param>
+            <param name="homed_position">1.22</param>
+            <param name="homing_kp">5.5</param>
+            <param name="homing_kd">0.2</param>
+            <param name="homing_torque_threshold">2.0</param>
+            <param name="position_min">-1.0</param>
+            <param name="position_max">1.0</param>
+            <param name="velocity_max">1.0</param>
+            <param name="effort_max">3.0</param>
+            <param name="kp_max">10.0</param>
+            <param name="kd_max">1.0</param>
+            <command_interface name="position"/>
+            <command_interface name="velocity"/>
+            <command_interface name="effort"/>
+            <command_interface name="kp"/>
+            <command_interface name="kd"/>
+            <state_interface name="position"/>
+            <state_interface name="velocity"/>
+        </joint>
+        <joint name="leg_back_l_2">
+            <param name="can_channel">3</param>
+            <param name="can_id">2</param>
+            <param name="homing_stage">1</param>
+            <param name="homing_velocity">1.0</param>
+            <param name="homed_position">0.42</param>
+            <param name="homing_kp">5.5</param>
+            <param name="homing_kd">0.2</param>
+            <param name="homing_torque_threshold">2.0</param>
+            <param name="position_min">-1.0</param>
+            <param name="position_max">1.0</param>
+            <param name="velocity_max">1.0</param>
+            <param name="effort_max">3.0</param>
+            <param name="kp_max">10.0</param>
+            <param name="kd_max">1.0</param>
+            <command_interface name="position"/>
+            <command_interface name="velocity"/>
+            <command_interface name="effort"/>
+            <command_interface name="kp"/>
+            <command_interface name="kd"/>
+            <state_interface name="position"/>
+            <state_interface name="velocity"/>
+        </joint>
+        <joint name="leg_back_l_3">
+            <param name="can_channel">3</param>
+            <param name="can_id">3</param>
+            <param name="homing_stage">0</param>
+            <param name="homing_velocity">-1.0</param>
+            <param name="homed_position">-0.62</param>
+            <param name="homing_kp">5.5</param>
+            <param name="homing_kd">0.2</param>
+            <param name="homing_torque_threshold">2.0</param>
+            <param name="position_min">-1.0</param>
+            <param name="position_max">1.0</param>
+            <param name="velocity_max">1.0</param>
+            <param name="effort_max">3.0</param>
+            <param name="kp_max">10.0</param>
+            <param name="kd_max">1.0</param>
+            <command_interface name="position"/>
+            <command_interface name="velocity"/>
+            <command_interface name="effort"/>
+            <command_interface name="kp"/>
+            <command_interface name="kd"/>
+            <state_interface name="position"/>
+            <state_interface name="velocity"/>
+        </joint>
         <joint name="leg_front_r_1">
             <param name="can_channel">2</param>
@@ -8,20 +146,20 @@
             <param name="homing_velocity">-1.0</param>
             <param name="homed_position">-1.22</param>
-            <param name="homing_kp">5.0</param>
-            <param name="homing_kd">0.2</param>
-            <param name="homing_torque_threshold">2.0</param>
-            <param name="position_min">-1.0</param>
-            <param name="position_max">1.0</param>
-            <param name="velocity_max">1.0</param>
-            <param name="effort_max">1.0</param>
-            <param name="kp_max">1.0</param>
-            <param name="kd_max">1.0</param>
-            <command_interface name="position" />
-            <command_interface name="velocity" />
-            <command_interface name="effort" />
-            <command_interface name="kp" />
-            <command_interface name="kd" />
-            <state_interface name="position" />
-            <state_interface name="velocity" />
+            <param name="homing_kp">5.5</param>
+            <param name="homing_kd">0.2</param>
+            <param name="homing_torque_threshold">2.0</param>
+            <param name="position_min">-1.0</param>
+            <param name="position_max">1.0</param>
+            <param name="velocity_max">1.0</param>
+            <param name="effort_max">3.0</param>
+            <param name="kp_max">10.0</param>
+            <param name="kd_max">1.0</param>
+            <command_interface name="position"/>
+            <command_interface name="velocity"/>
+            <command_interface name="effort"/>
+            <command_interface name="kp"/>
+            <command_interface name="kd"/>
+            <state_interface name="position"/>
+            <state_interface name="velocity"/>
         </joint>
         <joint name="leg_front_r_2">
@@ -31,20 +169,20 @@
             <param name="homing_velocity">-1.0</param>
             <param name="homed_position">-0.42</param>
-            <param name="homing_kp">5.0</param>
-            <param name="homing_kd">0.2</param>
-            <param name="homing_torque_threshold">2.0</param>
-            <param name="position_min">-1.0</param>
-            <param name="position_max">1.0</param>
-            <param name="velocity_max">1.0</param>
-            <param name="effort_max">1.0</param>
-            <param name="kp_max">1.0</param>
-            <param name="kd_max">1.0</param>
-            <command_interface name="position" />
-            <command_interface name="velocity" />
-            <command_interface name="effort" />
-            <command_interface name="kp" />
-            <command_interface name="kd" />
-            <state_interface name="position" />
-            <state_interface name="velocity" />
+            <param name="homing_kp">5.5</param>
+            <param name="homing_kd">0.2</param>
+            <param name="homing_torque_threshold">2.0</param>
+            <param name="position_min">-1.0</param>
+            <param name="position_max">1.0</param>
+            <param name="velocity_max">1.0</param>
+            <param name="effort_max">3.0</param>
+            <param name="kp_max">10.0</param>
+            <param name="kd_max">1.0</param>
+            <command_interface name="position"/>
+            <command_interface name="velocity"/>
+            <command_interface name="effort"/>
+            <command_interface name="kp"/>
+            <command_interface name="kd"/>
+            <state_interface name="position"/>
+            <state_interface name="velocity"/>
         </joint>
         <joint name="leg_front_r_3">
@@ -53,90 +191,21 @@
             <param name="homing_stage">0</param>
             <param name="homing_velocity">1.0</param>
-            <param name="homed_position">0.72</param>
-            <param name="homing_kp">5.0</param>
-            <param name="homing_kd">0.2</param>
-            <param name="homing_torque_threshold">2.0</param>
-            <param name="position_min">-1.0</param>
-            <param name="position_max">1.0</param>
-            <param name="velocity_max">1.0</param>
-            <param name="effort_max">1.0</param>
-            <param name="kp_max">1.0</param>
-            <param name="kd_max">1.0</param>
-            <command_interface name="position" />
-            <command_interface name="velocity" />
-            <command_interface name="effort" />
-            <command_interface name="kp" />
-            <command_interface name="kd" />
-            <state_interface name="position" />
-            <state_interface name="velocity" />
-        </joint>
-        <joint name="leg_front_l_1">
-            <param name="can_channel">1</param>
-            <param name="can_id">1</param>
-            <param name="homing_stage">2</param>
-            <param name="homing_velocity">1.0</param>
-            <param name="homed_position">1.22</param>
-            <param name="homing_kp">5.0</param>
-            <param name="homing_kd">0.2</param>
-            <param name="homing_torque_threshold">2.0</param>
-            <param name="position_min">-1.0</param>
-            <param name="position_max">1.0</param>
-            <param name="velocity_max">1.0</param>
-            <param name="effort_max">1.0</param>
-            <param name="kp_max">1.0</param>
-            <param name="kd_max">1.0</param>
-            <command_interface name="position" />
-            <command_interface name="velocity" />
-            <command_interface name="effort" />
-            <command_interface name="kp" />
-            <command_interface name="kd" />
-            <state_interface name="position" />
-            <state_interface name="velocity" />
-        </joint>
-        <joint name="leg_front_l_2">
-            <param name="can_channel">1</param>
-            <param name="can_id">2</param>
-            <param name="homing_stage">1</param>
-            <param name="homing_velocity">1.0</param>
-            <param name="homed_position">0.42</param>
-            <param name="homing_kp">5.0</param>
-            <param name="homing_kd">0.2</param>
-            <param name="homing_torque_threshold">2.0</param>
-            <param name="position_min">-1.0</param>
-            <param name="position_max">1.0</param>
-            <param name="velocity_max">1.0</param>
-            <param name="effort_max">1.0</param>
-            <param name="kp_max">1.0</param>
-            <param name="kd_max">1.0</param>
-            <command_interface name="position" />
-            <command_interface name="velocity" />
-            <command_interface name="effort" />
-            <command_interface name="kp" />
-            <command_interface name="kd" />
-            <state_interface name="position" />
-            <state_interface name="velocity" />
-        </joint>
-        <joint name="leg_front_l_3">
-            <param name="can_channel">1</param>
-            <param name="can_id">3</param>
-            <param name="homing_stage">0</param>
-            <param name="homing_velocity">-1.0</param>
-            <param name="homed_position">-0.72</param>
-            <param name="homing_kp">5.0</param>
-            <param name="homing_kd">0.2</param>
-            <param name="homing_torque_threshold">2.0</param>
-            <param name="position_min">-1.0</param>
-            <param name="position_max">1.0</param>
-            <param name="velocity_max">1.0</param>
-            <param name="effort_max">1.0</param>
-            <param name="kp_max">1.0</param>
-            <param name="kd_max">1.0</param>
-            <command_interface name="position" />
-            <command_interface name="velocity" />
-            <command_interface name="effort" />
-            <command_interface name="kp" />
-            <command_interface name="kd" />
-            <state_interface name="position" />
-            <state_interface name="velocity" />
+            <param name="homed_position">0.62</param>
+            <param name="homing_kp">5.5</param>
+            <param name="homing_kd">0.2</param>
+            <param name="homing_torque_threshold">2.0</param>
+            <param name="position_min">-1.0</param>
+            <param name="position_max">1.0</param>
+            <param name="velocity_max">1.0</param>
+            <param name="effort_max">3.0</param>
+            <param name="kp_max">10.0</param>
+            <param name="kd_max">1.0</param>
+            <command_interface name="position"/>
+            <command_interface name="velocity"/>
+            <command_interface name="effort"/>
+            <command_interface name="kp"/>
+            <command_interface name="kd"/>
+            <state_interface name="position"/>
+            <state_interface name="velocity"/>
         </joint>
         <joint name="leg_back_r_1">
@@ -146,20 +215,20 @@
             <param name="homing_velocity">-1.0</param>
             <param name="homed_position">-1.22</param>
-            <param name="homing_kp">5.0</param>
-            <param name="homing_kd">0.2</param>
-            <param name="homing_torque_threshold">2.0</param>
-            <param name="position_min">-1.0</param>
-            <param name="position_max">1.0</param>
-            <param name="velocity_max">1.0</param>
-            <param name="effort_max">1.0</param>
-            <param name="kp_max">1.0</param>
-            <param name="kd_max">1.0</param>
-            <command_interface name="position" />
-            <command_interface name="velocity" />
-            <command_interface name="effort" />
-            <command_interface name="kp" />
-            <command_interface name="kd" />
-            <state_interface name="position" />
-            <state_interface name="velocity" />
+            <param name="homing_kp">5.5</param>
+            <param name="homing_kd">0.2</param>
+            <param name="homing_torque_threshold">2.0</param>
+            <param name="position_min">-1.0</param>
+            <param name="position_max">1.0</param>
+            <param name="velocity_max">1.0</param>
+            <param name="effort_max">3.0</param>
+            <param name="kp_max">10.0</param>
+            <param name="kd_max">1.0</param>
+            <command_interface name="position"/>
+            <command_interface name="velocity"/>
+            <command_interface name="effort"/>
+            <command_interface name="kp"/>
+            <command_interface name="kd"/>
+            <state_interface name="position"/>
+            <state_interface name="velocity"/>
         </joint>
         <joint name="leg_back_r_2">
@@ -169,20 +238,20 @@
             <param name="homing_velocity">-1.0</param>
             <param name="homed_position">-0.42</param>
-            <param name="homing_kp">5.0</param>
-            <param name="homing_kd">0.2</param>
-            <param name="homing_torque_threshold">2.0</param>
-            <param name="position_min">-1.0</param>
-            <param name="position_max">1.0</param>
-            <param name="velocity_max">1.0</param>
-            <param name="effort_max">1.0</param>
-            <param name="kp_max">1.0</param>
-            <param name="kd_max">1.0</param>
-            <command_interface name="position" />
-            <command_interface name="velocity" />
-            <command_interface name="effort" />
-            <command_interface name="kp" />
-            <command_interface name="kd" />
-            <state_interface name="position" />
-            <state_interface name="velocity" />
+            <param name="homing_kp">5.5</param>
+            <param name="homing_kd">0.2</param>
+            <param name="homing_torque_threshold">2.0</param>
+            <param name="position_min">-1.0</param>
+            <param name="position_max">1.0</param>
+            <param name="velocity_max">1.0</param>
+            <param name="effort_max">3.0</param>
+            <param name="kp_max">10.0</param>
+            <param name="kd_max">1.0</param>
+            <command_interface name="position"/>
+            <command_interface name="velocity"/>
+            <command_interface name="effort"/>
+            <command_interface name="kp"/>
+            <command_interface name="kd"/>
+            <state_interface name="position"/>
+            <state_interface name="velocity"/>
         </joint>
         <joint name="leg_back_r_3">
@@ -191,90 +260,21 @@
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